File: PowerManagement.kicad_sch (KiCad schematic)
At the start: 22 parts, among them J5 Screw_Terminal_01x02_POWER, U2 XC6210B332MR, U3 XL1509

Commit message: more layout
Connections:
- net +3.3V: now also R3.1; no longer D5.2
- net GND: now also D5.1; no longer R3.2
- new net: D5.2, R3.2
Other:
- moved on the sheet: D5, R3
Changed lines of the file:
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@@
 	(symbol
 		(lib_id "PCM_JLCPCB-Diodes:LED,0603,Yellow")
-		(at 182.88 100.33 0)
+		(at 182.88 110.49 0)
 		(unit 1)
 		(exclude_from_sim no)
@@
 		(fields_autoplaced yes)
 		(property "Reference" "D5"
-			(at 185.42 98.9646 0)
+			(at 185.42 109.1246 0)
 			(effects
 				(font
@@
 		)
 		(property "Value" "Yellow"
-			(at 185.42 101.5047 0)
+			(at 185.42 111.6647 0)
 			(effects
 				(font
@@
 		)
 		(property "Footprint" "PCM_JLCPCB:D_0603"
-			(at 181.102 100.33 90)
+			(at 181.102 110.49 90)
 			(effects
 				(font
@@
 		)
 		(property "Datasheet" "https://www.lcsc.com/datasheet/lcsc_datasheet_2008201033_Foshan-NationStar-Optoelectronics-NCD0603Y2_C89811.pdf"
-			(at 182.88 100.33 0)
+			(at 182.88 110.49 0)
 			(effects
 				(font
@@
 		)
 		(property "Description" "25mA 100mcd~220mcd Colorless transparent lens 586nm~595nm -30°C~+85°C Yellow 130° 65mW 1.6V~2.6V 0603 LED Indication - Discrete ROHS"
-			(at 182.88 100.33 0)
+			(at 182.88 110.49 0)
 			(effects
 				(font
@@
 		)
 		(property "LCSC" "C89811"
-			(at 182.88 100.33 0)
+			(at 182.88 110.49 0)
 			(effects
 				(font
@@
 		)
 		(property "Stock" "109176"
-			(at 182.88 100.33 0)
+			(at 182.88 110.49 0)
 			(effects
 				(font
@@
 		)
 		(property "Price" "0.021USD"
-			(at 182.88 100.33 0)
+			(at 182.88 110.49 0)
 			(effects
 				(font
@@
 		)
 		(property "Process" "SMT"
-			(at 182.88 100.33 0)
+			(at 182.88 110.49 0)
 			(effects
 				(font
@@
 		)
 		(property "Minimum Qty" "20"
-			(at 182.88 100.33 0)
+			(at 182.88 110.49 0)
 			(effects
 				(font
@@
 		)
 		(property "Attrition Qty" "6"
-			(at 182.88 100.33 0)
+			(at 182.88 110.49 0)
 			(effects
 				(font
@@
 		)
 		(property "Class" "Preferred Component"
-			(at 182.88 100.33 0)
+			(at 182.88 110.49 0)
 			(effects
 				(font
@@
 		)
 		(property "Category" "Optoelectronics,Light Emitting Diodes (LED)"
-			(at 182.88 100.33 0)
+			(at 182.88 110.49 0)
 			(effects
 				(font
@@
 		)
 		(property "Manufacturer" "Foshan NationStar Optoelectronics"
-			(at 182.88 100.33 0)
+			(at 182.88 110.49 0)
 			(effects
 				(font
@@
 		)
 		(property "Part" "NCD0603Y2"
-			(at 182.88 100.33 0)
+			(at 182.88 110.49 0)
 			(effects
 				(font
@@
 		)
 		(property "Dominant Wavelength" "586nm~595nm"
-			(at 182.88 100.33 0)
+			(at 182.88 110.49 0)
 			(effects
 				(font
@@
 		)
 		(property "Operating Temperature" "-30°C~+85°C"
-			(at 182.88 100.33 0)
+			(at 182.88 110.49 0)
 			(effects
 				(font
@@
 		)
 		(property "Power Dissipation" "65mW"
-			(at 182.88 100.33 0)
+			(at 182.88 110.49 0)
 			(effects
 				(font
@@
 		)
 		(property "Emitted Color" "Yellow"
-			(at 182.88 100.33 0)
+			(at 182.88 110.49 0)
 			(effects
 				(font
@@
 		)
 		(property "Viewing Angle" "130°"
-			(at 182.88 100.33 0)
+			(at 182.88 110.49 0)
 			(effects
 				(font
@@
 		)
 		(property "Forward Current" "25mA"
-			(at 182.88 100.33 0)
+			(at 182.88 110.49 0)
 			(effects
 				(font
@@
 		)
 		(property "Forward Voltage (VF)" "1.6V~2.6V"
-			(at 182.88 100.33 0)
+			(at 182.88 110.49 0)
 			(effects
 				(font
@@
 		)
 		(property "Lens Color" "Colorless Transparent Lens"
-			(at 182.88 100.33 0)
+			(at 182.88 110.49 0)
 			(effects
 				(font
@@
 		)
 		(property "Luminous Intensity" "100mcd~220mcd"
-			(at 182.88 100.33 0)
+			(at 182.88 110.49 0)
 			(effects
 				(font
@@
 	(symbol
 		(lib_id "PCM_JLCPCB-Resistors:0603,1kΩ")
-		(at 182.88 110.49 0)
+		(at 182.88 100.33 0)
 		(unit 1)
 		(exclude_from_sim no)
@@
 		(dnp no)
 		(property "Reference" "R3"
-			(at 185.166 110.49 90)
+			(at 185.166 100.33 90)
 			(effects
 				(font
@@
 		)
 		(property "Value" "1kΩ"
-			(at 182.88 110.49 90)
+			(at 182.88 100.33 90)
 			(do_not_autoplace yes)
 			(effects
@@
 		)
 		(property "Footprint" "PCM_JLCPCB:R_0603"
-			(at 181.102 110.49 90)
+			(at 181.102 100.33 90)
 			(effects
 				(font
@@
 		)
 		(property "Datasheet" "https://www.lcsc.com/datasheet/lcsc_datasheet_2206010130_UNI-ROYAL-Uniroyal-Elec-0603WAF1001T5E_C21190.pdf"
-			(at 182.88 110.49 0)
+			(at 182.88 100.33 0)
 			(effects
 				(font
@@
 		)
 		(property "Description" "100mW Thick Film Resistors 75V ±100ppm/°C ±1% 1kΩ 0603 Chip Resistor - Surface Mount ROHS"
-			(at 182.88 110.49 0)
+			(at 182.88 100.33 0)
 			(effects
 				(font
@@
 		)
 		(property "LCSC" "C21190"
-			(at 182.88 110.49 0)
+			(at 182.88 100.33 0)
 			(effects
 				(font
@@
 		)
 		(property "Stock" "27538425"
-			(at 182.88 110.49 0)
+			(at 182.88 100.33 0)
 			(effects
 				(font
@@
 		)
 		(property "Price" "0.004USD"
-			(at 182.88 110.49 0)
+			(at 182.88 100.33 0)
 			(effects
 				(font
@@
 		)
 		(property "Process" "SMT"
-			(at 182.88 110.49 0)
+			(at 182.88 100.33 0)
 			(effects
 				(font
@@
 		)
 		(property "Minimum Qty" "20"
-			(at 182.88 110.49 0)
+			(at 182.88 100.33 0)
 			(effects
 				(font
@@
 		)
 		(property "Attrition Qty" "10"
-			(at 182.88 110.49 0)
+			(at 182.88 100.33 0)
 			(effects
 				(font
@@
 		)
 		(property "Class" "Basic Component"
-			(at 182.88 110.49 0)
+			(at 182.88 100.33 0)
 			(effects
 				(font
@@
 		)
 		(property "Category" "Resistors,Chip Resistor - Surface Mount"
-			(at 182.88 110.49 0)
+			(at 182.88 100.33 0)
 			(effects
 				(font
@@
 		)
 		(property "Manufacturer" "UNI-ROYAL(Uniroyal Elec)"
-			(at 182.88 110.49 0)
+			(at 182.88 100.33 0)
 			(effects
 				(font
@@
 		)
 		(property "Part" "0603WAF1001T5E"
-			(at 182.88 110.49 0)
+			(at 182.88 100.33 0)
 			(effects
 				(font
@@
 		)
 		(property "Resistance" "1kΩ"
-			(at 182.88 110.49 0)
+			(at 182.88 100.33 0)
 			(effects
 				(font
@@
 		)
 		(property "Power(Watts)" "100mW"
-			(at 182.88 110.49 0)
+			(at 182.88 100.33 0)
 			(effects
 				(font
@@
 		)
 		(property "Type" "Thick Film Resistors"
-			(at 182.88 110.49 0)
+			(at 182.88 100.33 0)
 			(effects
 				(font
@@
 		)
 		(property "Overload Voltage (Max)" "75V"
-			(at 182.88 110.49 0)
+			(at 182.88 100.33 0)
 			(effects
 				(font
@@
 		)
 		(property "Operating Temperature Range" "-55°C~+155°C"
-			(at 182.88 110.49 0)
+			(at 182.88 100.33 0)
 			(effects
 				(font
@@
 		)
 		(property "Tolerance" "±1%"
-			(at 182.88 110.49 0)
+			(at 182.88 100.33 0)
 			(effects
 				(font
@@
 		)
 		(property "Temperature Coefficient" "±100ppm/°C"
-			(at 182.88 110.49 0)
+			(at 182.88 100.33 0)
 			(effects
 				(font
