File: Encoder.kicad_sch (KiCad schematic)
At the start: 20 parts, among them J4 C225127, J7 C225127, U5 AS5047D

Commit message: Placement, some layout
Parts:
- added U8: AS5047D, Package_SO:TSSOP-14_4.4x5mm_P0.65mm, symbol Sensor_Magnetic:AS5047D
Other:
- note added: "Dummy Footprint. (To get the encoder placed on the front side)"
