File: Mcu.kicad_sch (KiCad schematic)
At the start: 68 parts, among them J10 AUX2, J14 IO, J15 IO, J16 IO, J17 IO, J18 IO, J19 IO, J20 IO, J21 IO, J22 IO, J23 IO, J24 IO, J25 IO, J26 IO, J27 IO, J28 IO, J29 IO, J30 IO, J31 IO, J32 IO, J33 IO, J34 IO, J35 IO, J36 IO, J37 IO, J38 IO, J39 IO, J40 IO, J41 IO, J42 IO, J43 IO, J44 IO, J45 IO, J46 IO, J47 IO, J48 IO, J49 IO, J50 IO, J51 IO, J52 IO, J53 IO, J54 IO, J55 IO, J56 IO, U12 STM32H723VGT6, X2 X322516MLB4SI

Commit message: layout fine tuning
Connections:
- net DEBUG_RX: now also J54.1 (Pin_1)
- net DEBUG_TX: now also J55.1 (Pin_1)
Changed lines of the file:
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@@
 		)
 	)
+	(global_label "DEBUG_TX"
+		(shape input)
+		(at 152.4 21.59 180)
+		(fields_autoplaced yes)
+		(effects
+			(font
+				(size 1.016 1.016)
+				(color 255 200 0 1)
+			)
+			(justify right)
+		)
+		(property "Intersheetrefs" "${INTERSHEET_REFS}"
+			(at 142.4647 21.59 0)
+			(hide yes)
+			(show_name no)
+			(do_not_autoplace no)
+			(effects
+				(font
+					(size 1.27 1.27)
+				)
+				(justify right)
+			)
+		)
+	)
 	(global_label "DRV_SPI_~{SCS}"
 		(shape input)
@@
 		)
 	)
+	(global_label "DEBUG_RX"
+		(shape input)
+		(at 152.4 17.78 180)
+		(fields_autoplaced yes)
+		(effects
+			(font
+				(size 1.016 1.016)
+				(color 255 200 0 1)
+			)
+			(justify right)
+		)
+		(property "Intersheetrefs" "${INTERSHEET_REFS}"
+			(at 142.2228 17.78 0)
+			(hide yes)
+			(show_name no)
+			(do_not_autoplace no)
+			(effects
+				(font
+					(size 1.27 1.27)
+				)
+				(justify right)
+			)
+		)
+	)
 	(global_label "RS485_DI"
 		(shape output)
@@
 	)
 	(symbol
+		(lib_id "Connector_Generic:Conn_01x01")
+		(at 73.66 17.78 0)
+		(unit 1)
+		(body_style 1)
+		(exclude_from_sim no)
+		(in_bom yes)
+		(on_board yes)
+		(in_pos_files yes)
+		(dnp no)
+		(property "Reference" "J56"
+			(at 76.962 17.78 0)
+			(show_name no)
+			(do_not_autoplace no)
+			(effects
+				(font
+					(size 1.27 1.27)
+				)
+				(justify left)
+			)
+		)
+		(property "Value" "IO"
+			(at 74.93 17.78 0)
+			(show_name no)
+			(do_not_autoplace no)
+			(effects
+				(font
+					(size 1.27 1.27)
+				)
+				(justify left)
+			)
+		)
+		(property "Footprint" "TestPoint:TestPoint_THTPad_D1.0mm_Drill0.5mm"
+			(at 73.66 17.78 0)
+			(hide yes)
+			(show_name no)
+			(do_not_autoplace no)
+			(effects
+				(font
+					(size 1.27 1.27)
+				)
+			)
+		)
+		(property "Datasheet" ""
+			(at 73.66 17.78 0)
+			(hide yes)
+			(show_name no)
+			(do_not_autoplace no)
+			(effects
+				(font
+					(size 1.27 1.27)
+				)
+			)
+		)
+		(property "Description" "Generic connector, single row, 01x01, script generated (kicad-library-utils/schlib/autogen/connector/)"
+			(at 73.66 17.78 0)
+			(hide yes)
+			(show_name no)
+			(do_not_autoplace no)
+			(effects
+				(font
+					(size 1.27 1.27)
+				)
+			)
+		)
+		(pin "1"
+		)
+		(instances
+			(project "PiccoloMotorDriver"
+				(path "/cc8a13e7-b1a6-4cbd-adcd-4feb8b2e2369/18750508-a205-46c6-b741-330bfb864ed8"
+					(reference "J56")
+					(unit 1)
+				)
+			)
+		)
+	)
+	(symbol
 		(lib_id "PCM_JLCPCB-Capacitors:0603,10pF")
 		(at 341.63 165.1 0)
@@
 					(unit 1)
 				)
-			)
-		)
-	)
-	(symbol
-		(lib_id "Connector_Generic:Conn_01x01")
-		(at 73.66 17.78 0)
-		(unit 1)
-		(body_style 1)
-		(exclude_from_sim no)
-		(in_bom yes)
-		(on_board yes)
-		(in_pos_files yes)
-		(dnp no)
-		(property "Reference" "J56"
-			(at 76.962 17.78 0)
-			(show_name no)
-			(do_not_autoplace no)
-			(effects
-				(font
-					(size 1.27 1.27)
-				)
-				(justify left)
-			)
-		)
-		(property "Value" "IO"
-			(at 74.93 17.78 0)
-			(show_name no)
-			(do_not_autoplace no)
-			(effects
-				(font
-					(size 1.27 1.27)
-				)
-				(justify left)
-			)
-		)
-		(property "Footprint" "TestPoint:TestPoint_THTPad_D1.0mm_Drill0.5mm"
-			(at 73.66 17.78 0)
-			(hide yes)
-			(show_name no)
-			(do_not_autoplace no)
-			(effects
-				(font
-					(size 1.27 1.27)
-				)
-			)
-		)
-		(property "Datasheet" ""
-			(at 73.66 17.78 0)
-			(hide yes)
-			(show_name no)
-			(do_not_autoplace no)
-			(effects
-				(font
-					(size 1.27 1.27)
-				)
-			)
-		)
-		(property "Description" "Generic connector, single row, 01x01, script generated (kicad-library-utils/schlib/autogen/connector/)"
-			(at 73.66 17.78 0)
-			(hide yes)
-			(show_name no)
-			(do_not_autoplace no)
-			(effects
-				(font
-					(size 1.27 1.27)
-				)
-			)
-		)
-		(pin "1"
-		)
-		(instances
-			(project "PiccoloMotorDriver"
-				(path "/cc8a13e7-b1a6-4cbd-adcd-4feb8b2e2369/18750508-a205-46c6-b741-330bfb864ed8"
-					(reference "J56")
-					(unit 1)
-				)

Commit message: DRC check - fine tuning
Parts:
- removed J10: AUX2, Connector_PinSocket_2.54mm:PinSocket_2x03_P2.54mm_Vertical, symbol Connector_Generic:Conn_02x03_Odd_Even
- added J58: IO, TestPoint:TestPoint_THTPad_D1.0mm_Drill0.5mm, symbol Connector_Generic:Conn_01x01
Connections:
- net DRV_OFF renamed DRV_ENABLE
- net ~{DRV_SLEEP} renamed PB2
- net PB2: now also J58.1 (Pin_1)
Other:
- moved on the sheet: J25, J26, J27, J28, J29, J30, J31, J32

Commit message: Drc, Bom done
Parts:
- U12: LCSC (none) -> C730142
Changed lines of the file:
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@@
 			)
 		)
+		(property "LCSC" "C730142"
+			(at 102.362 230.378 0)
+			(effects
+				(font
+					(size 1.27 1.27)
+				)
+				(hide yes)
+			)
+		)
 		(pin "27"
 		)
@@
 			)
 		)
+		(property "LCSC" "C730142"
+			(at 268.224 57.912 0)
+			(effects
+				(font
+					(size 1.27 1.27)
+				)
+				(hide yes)
+			)
+		)
 		(pin "27"
 		)
@@
 			)
 		)
+		(property "LCSC" "C730142"
+			(at 269.494 151.892 0)
+			(effects
+				(font
+					(size 1.27 1.27)
+				)
+				(hide yes)
+			)
+		)
