File: IO.kicad_sch (KiCad schematic)
At the start: 20 parts, among them J1 Conn_01x06_SWD, J11 C189893, J3 C189893, J6 Connector, USB-TYPE-C-16P, SW1 SW_DIP_x02, U1 SP485EEN, U4 TJA1050T/CM,118, U6 USBLC6-2SC6

Commit message: Replaced 3.3V linear regulator with switch mode regulator
Parts:
- added JP1: RS485, Jumper:SolderJumper-2_P1.3mm_Open_TrianglePad1.0x1.5mm, symbol Jumper:SolderJumper_2_Open
- added JP2: CAN, Jumper:SolderJumper-2_P1.3mm_Open_TrianglePad1.0x1.5mm, symbol Jumper:SolderJumper_2_Open
Connections:
- net CAN-: now also JP2.1 (A)
- net RS485+: now also JP1.2 (B)
- net can_termination_B: now also JP2.2 (B)
- net rs485_termination_B: now also JP1.1 (A)
